File: kicad/node_monitor/node_monitor/node_monitor.sch (KiCad schematic (older format))
At the start: 16 parts

Commit message: 158
Parts:
- removed J?: Conn_01x02_Male, symbol Connector:Conn_01x02_Male
- added J3: Conn_01x03_Male, Connector_PinHeader_2.54mm:PinHeader_1x03_P2.54mm_Vertical, symbol Connector:Conn_01x03_Male
- added J8: Conn_01x02_Male, Connector_PinHeader_2.54mm:PinHeader_1x02_P2.54mm_Vertical, symbol Connector:Conn_01x02_Male
- B1: renamed from B?; footprint (none) -> custom:BLUEPILL
- C1, C2: renamed from C?; footprint (none) -> Capacitor_THT:CP_Radial_D5.0mm_P2.50mm
- J1, J2, J5: renamed from J?; footprint (none) -> Connector_PinHeader_2.54mm:PinHeader_1x02_P2.54mm_Vertical
- J4: renamed from J?; footprint (none) -> Connector_RJ:RJ45_Ninigi_GE
- J6, J7: renamed from J?; footprint (none) -> Connector_PinHeader_2.54mm:PinHeader_1x03_P2.54mm_Vertical
- L1: renamed from L?; footprint (none) -> custom:LM2596
- L2: renamed from L?; footprint (none) -> custom:LORA
- R1: renamed from R?; footprint (none) -> custom:RS485
- R2, R3: renamed from R?; footprint (none) -> Resistor_THT:R_Axial_DIN0204_L3.6mm_D1.6mm_P7.62mm_Horizontal
- SW1: renamed from SW?; footprint (none) -> Package_DIP:DIP-12_W7.62mm
Connections:
- net GND is gone; now on net GND1: C1.2, C2.2, J6.3 (Pin_3), J7.3 (Pin_3), L1.4 (VOUT-)
- net GND2 is gone; now on net GND1: B1.40 (GND), L2.7 (GND)
- net 3V3: now also B1.20 (3V3), SW1.10, SW1.11; no longer SW1.2, SW1.3
- net A: now also J4.3, J4.4
- net AUX: now also B1.32 (PA7); no longer B1.26 (PA1)
- net B: now also J4.5, J4.6
- net GND1: now also J4.7, J4.8, J3.3 (Pin_3)
- net LRXD: now also SW1.8, J8.1 (Pin_1); no longer SW1.6
- net LRXI: now also SW1.5; no longer SW1.7
- net LTXD: now also SW1.7, J8.2 (Pin_2); no longer SW1.5
- net LTXI: now also SW1.6; no longer SW1.8
- net VCCI: now also SW1.1; no longer SW1.12
- net VCCO: now also SW1.12; no longer SW1.1
- net RLI: now reaches B1.29 (PA4)
- net RLI: now also SW1.4
- net MANUAL: now reaches B1.30 (PA5)
- net MANUAL: now also SW1.3
- net MODE: now reaches B1.31 (PA6)
- net MODE: now also SW1.2
- net RLD: now reaches SW1.9
- net RLD: now also J3.2 (Pin_2)
- net at R2.2: now also J3.1 (Pin_1)

Commit message: 3698
Other:
- moved on the sheet: B1, C1, C2, J1, J2, J3, J5, J6, J7, J8, L1, L2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
